Commit message: Add files via upload

File: backwards_knee.urdf (robot description, URDF)
Before this commit: robot backwards_knee, 7 links, 7 joints
Links:
- added link toe
- link body: geometry collision sphere radius=0.35; visual sphere radius=0.35
- link foot: geometry collision cylinder length=0.12 radius=0.015; visual cylinder length=0.12 radius=0.015
- link lower leg: geometry collision cylinder length=0.12 radius=0.015; visual cylinder length=0.12 radius=0.015
Joints:
- added joint toe_pos: type fixed, parent foot, child toe, origin xyz=0.82 0 -0.30
- joint ankle: origin xyz=0 0 0.012 -> xyz=-0.48 0 -0.82
- joint hip: origin xyz=0 0 0.094 -> xyz=0 0 -0.35
- joint knee: origin xyz=0 0 0.06 -> xyz=0.39 0 -0.13 rpy=0 0 0

Commit message: Add files via upload

File: backwards_knee.urdf (robot description, URDF)
Before this commit: robot backwards_knee, 8 links, 8 joints
Links:
- removed link toe
Joints:
- removed joint toe_pos

Commit message: Add files via upload

File: backwards_knee.urdf (robot description, URDF)
Before this commit: robot backwards_knee, 7 links, 7 joints
Links:
- link body: geometry collision sphere radius=0.35; visual sphere radius=0.1

Commit message: Add files via upload

File: backwards_knee.urdf (robot description, URDF)
Before this commit: robot backwards_knee, 7 links, 7 joints
Links:
- link foot: geometry collision cylinder length=0.9 radius=0.015; visual cylinder length=0.9 radius=0.15
- link lower leg: geometry collision cylinder length=0.96 radius=0.15; visual cylinder length=0.96 radius=0.15
- link upper leg: geometry collision cylinder length=0.38 radius=0.15; visual cylinder length=0.38 radius=0.15

Commit message: Add files via upload

File: backwards_knee.urdf (robot description, URDF)
Before this commit: robot backwards_knee, 7 links, 7 joints
Links:
- link body: mass 1 -> .1; geometry collision sphere radius=0.35; visual sphere radius=0.35

Commit message: Add files via upload

File: backwards_knee.urdf (robot description, URDF)
Before this commit: robot backwards_knee, 7 links, 7 joints
Links:
- link foot: geometry collision cylinder length=0.9 radius=0.05; visual cylinder length=0.9 radius=0.05
- link lower leg: geometry collision cylinder length=0.96 radius=0.05; visual cylinder length=0.96 radius=0.05
- link upper leg: geometry collision cylinder length=0.38 radius=0.05; visual cylinder length=0.38 radius=0.05

Commit message: Add files via upload

File: backwards_knee.urdf (robot description, URDF)
Before this commit: robot backwards_knee, 7 links, 7 joints
Links:
- link body: geometry collision sphere radius=0.35; visual sphere radius=0.35
- link foot: geometry collision cylinder length=0.96 radius=0.05; visual cylinder length=0.96 radius=0.05
- link upper leg: geometry collision cylinder length=0.4 radius=0.05; visual cylinder length=0.4 radius=0.05
Joints:
- joint ankle: origin xyz=-0.48 0 -0.82 -> xyz=0.48 0 -0.82
- joint ground_to_dummy1: origin xyz=0 0 0 -> xyz=0 0 1
- joint knee: origin xyz=0.39 0 -0.13 rpy=0 0 0 -> xyz=-0.14 0 -0.38 rpy=0 0 0

Commit message: Add files via upload

File: backwards_knee.urdf (robot description, URDF)
Before this commit: robot backwards_knee, 7 links, 7 joints
Joints:
- joint hip: origin xyz=0 0 -0.35 -> xyz=0 0 0

Commit message: Add files via upload

File: backwards_knee.urdf (robot description, URDF)
Before this commit: robot backwards_knee, 7 links, 7 joints
Links:
- removed link foot
Joints:
- removed joint ankle

Commit message: Add files via upload

File: backwards_knee.urdf (robot description, URDF)
Before this commit: robot backwards_knee, 6 links, 6 joints
Links:
- added link foot, mass .1; collision cylinder length=0.96 radius=0.05; visual cylinder length=0.96 radius=0.05
Joints:
- added joint ankle: type revolute, parent lower leg, child foot, origin xyz=0.48 0 -0.82, axis 0 1 0, limit lower=-3.14 upper=0 effort=100 velocity=1.57

Commit message: Add files via upload

File: backwards_knee.urdf (robot description, URDF)
Before this commit: robot backwards_knee, 7 links, 7 joints
Joints:
- joint hip: origin xyz=0 0 0 -> xyz=0 0 -0.35

Commit message: Add files via upload

File: backwards_knee.urdf (robot description, URDF)
Before this commit: robot backwards_knee, 7 links, 7 joints
Joints:
- joint ankle: origin xyz=0.48 0 -0.82 -> xyz=0 0 0
- joint knee: origin xyz=-0.14 0 -0.38 rpy=0 0 0 -> xyz=0 0 0 rpy=0 0 0

Commit message: Add files via upload

File: backwards_knee.urdf (robot description, URDF)
Before this commit: robot backwards_knee, 7 links, 7 joints
Joints:
- joint ground_to_dummy1: origin xyz=0 0 1 -> xyz=0 0 2

Commit message: Add files via upload

File: backwards_knee.urdf (robot description, URDF)
Before this commit: robot backwards_knee, 7 links, 7 joints
Joints:
- joint knee: origin xyz=0 0 0 rpy=0 0 0 -> xyz=-0.14 0 -0.38 rpy=0 0 0

Commit message: Add files via upload

File: backwards_knee.urdf (robot description, URDF)
Before this commit: robot backwards_knee, 7 links, 7 joints
Links:
- link foot: geometry collision cylinder length=0.92 radius=0.05; visual cylinder length=0.92 radius=0.05
Joints:
- joint ankle: origin xyz=0 0 0 -> xyz=0 0 -0.96
- joint knee: origin xyz=-0.14 0 -0.38 rpy=0 0 0 -> xyz=0 0 -0.4 rpy=0 0 0

Commit message: Add files via upload

File: backwards_knee.urdf (robot description, URDF)
Before this commit: robot backwards_knee, 7 links, 7 joints
Joints:
- joint ground_to_dummy1: origin xyz=0 0 3 -> xyz=0 0 4

Commit message: Add files via upload

File: backwards_knee.urdf (robot description, URDF)
Before this commit: robot backwards_knee, 7 links, 7 joints
Joints:
- joint ankle: axis 0 1 0 -> 0 -1 0
- joint hip: axis 0 1 0 -> 0 -1 0
- joint knee: axis 0 1 0 -> 0 -1 0

Commit message: Add files via upload

File: backwards_knee.urdf (robot description, URDF)
Before this commit: robot backwards_knee, 7 links, 7 joints
Joints:
- joint ankle: limit lower=-3.14 upper=0 effort=100 velocity=1.57 -> lower=-1.57 upper=1.57 effort=100 velocity=1.57
- joint hip: limit lower=-3.14 upper=0 effort=100 velocity=1.57 -> lower=-1.57 upper=1.57 effort=100 velocity=1.57
